File: kicad_4l60e/kicad_4l60e.kicad_sch (KiCad schematic)
At the start: 78 parts, among them IC1 LM2903P, J1 DC37_Socket, J2 Conn_01x01_Pin, J3 Conn_01x01_Pin, J4 Conn_01x01_Pin, J5 Conn_01x01_Pin, Q1 STP36NF06L, Q2 STP36NF06L, Q3 STP36NF06L, Q4 STP36NF06L, U1 Teensy4.1

Commit message: updates
Other:
- added sheet Case Connectors (case_connectors.kicad_sch)
- added sheet Comms (comms.kicad_sch)
- added sheet EPC Driver (epc_driver.kicad_sch)
- added sheet Inputs (inputs.kicad_sch)
- added sheet Power Supply (power_supply.kicad_sch)
- added sheet Raspberry Pi Zero 2W (pi_zero_2w.kicad_sch)
- added sheet Solenoid Drivers (solenoid_drivers.kicad_sch)
- added sheet Teensy 4.1 (teensy_4.1.kicad_sch)
- added sheet VSS VR Conditioner (vss_vr_conditioner.kicad_sch)
