File: kicad_4l60e/individual_schematics/4l60e_input_pressure_switch_manifold.kicad_sch (KiCad schematic)
At the start: 3 parts

Commit message: updates
Changed lines of the file:
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@@
 	(text "PRESSURE SWITCH MANIFOLD (Pins 20/21/22)\nGear confirmation A/B/C\n10k pullups, ground-switched (active LOW)\nJ6: pin1=A, pin2=B, pin3=C, pin4=GND"
 		(exclude_from_sim no)
-		(at 126.492 51.054 0)
+		(at 122.174 58.928 0)
 		(effects
 			(font
@@
 	(text "Pin A: TFP Switch 3"
 		(exclude_from_sim no)
-		(at 40.64 64.262 0)
+		(at 81.28 64.262 0)
 		(effects
 			(font
@@
 	(text "To Teensy 4.1 Pin 21"
 		(exclude_from_sim no)
-		(at 127.762 74.168 0)
+		(at 127.762 72.898 0)
 		(effects
 			(font
@@
 	(text "Pin A: TFP Switch 2"
 		(exclude_from_sim no)
-		(at 40.386 59.436 0)
+		(at 81.026 59.436 0)
 		(effects
 			(font
@@
 	(text "To Teensy 4.1 Pin 20"
 		(exclude_from_sim no)
-		(at 112.268 82.296 0)
+		(at 112.268 78.486 0)
 		(effects
 			(font
@@
 	(text "Pin A: TFP Switch 1"
 		(exclude_from_sim no)
-		(at 40.132 53.594 0)
+		(at 80.772 53.594 0)
 		(effects
 			(font
@@
 	(wire
 		(pts
-			(xy 27.94 60.96) (xy 110.49 60.96)
-		)
-		(stroke
-			(width 0)
-			(type default)
-		)
-	)
-	(wire
-		(pts
-			(xy 100.33 55.88) (xy 100.33 80.01)
+			(xy 68.58 60.96) (xy 110.49 60.96)
+		)
+		(stroke
+			(width 0)
+			(type default)
+		)
+	)
+	(wire
+		(pts
+			(xy 100.33 55.88) (xy 100.33 76.2)
 		)
 		(stroke
@@
 	(wire
 		(pts
-			(xy 29.21 55.88) (xy 100.33 55.88)
-		)
-		(stroke
-			(width 0)
-			(type default)
-		)
-	)
-	(wire
-		(pts
-			(xy 100.33 80.01) (xy 124.46 80.01)
+			(xy 69.85 55.88) (xy 100.33 55.88)
+		)
+		(stroke
+			(width 0)
+			(type default)
+		)
+	)
+	(wire
+		(pts
+			(xy 100.33 76.2) (xy 124.46 76.2)
 		)
 		(stroke
@@
 	(wire
 		(pts
-			(xy 26.67 66.04) (xy 120.65 66.04)
+			(xy 67.31 66.04) (xy 120.65 66.04)
 		)
 		(stroke
@@
 	(wire
 		(pts
-			(xy 110.49 60.96) (xy 110.49 72.39)
-		)
-		(stroke
-			(width 0)
-			(type default)
-		)
-	)
-	(wire
-		(pts
-			(xy 110.49 72.39) (xy 135.89 72.39)
-		)
-		(stroke
+			(xy 110.49 60.96) (xy 110.49 71.12)
+		)
+		(stroke
+			(width 0)
+			(type default)
+		)
+	)
+	(wire
+		(pts
+			(xy 110.49 71.12) (xy 135.89 71.12)
+		)
+		(stroke
